File: Switchboard.sch (KiCad schematic (older format))
At the start: 16 parts, among them J2 Conn_01x02_Female, J3 AudioJack2_SwitchT, J4 Conn_01x06_Female, J5 AudioJack2_SwitchT, SW1 SW_3PDT_x3, U101 LTC1044

Commit message: Tweak some resistor values
Parts:
- R101: value 1k -> 100
Changed lines of the file:
@@
 Sheet 1 1
 Title "Switchboard"
-Date "2019-11-03"
-Rev "r01"
+Date "2020-12-30"
+Rev "r02"
 Comp "Nuclear Lighthouse Studios"
 Comment1 "CC BY-NC-SA"
@@
 P 5000 5900
 F 0 "R101" H 4930 5854 50  0000 R CNN
-F 1 "1k" H 4930 5945 50  0000 R CNN
+F 1 "100" H 4930 5945 50  0000 R CNN
 F 2 "Resistor_THT:R_Axial_DIN0207_L6.3mm_D2.5mm_P2.54mm_Vertical" V 4930 5900 50  0001 C CNN
 F 3 "~" H 5000 5900 50  0001 C CNN
@@
 	5000 6400 5050 6400
 $Comp
-L power:PWR_FLAG #FLG?
+L power:PWR_FLAG #FLG0102
 U 1 1 5D696FAB
 P 2700 2450
-F 0 "#FLG?" H 2700 2525 50  0001 C CNN
+F 0 "#FLG0102" H 2700 2525 50  0001 C CNN
 F 1 "PWR_FLAG" V 2700 2577 50  0000 L CNN
 F 2 "" H 2700 2450 50  0001 C CNN
