File: Switchboard.kicad_pcb (KiCad board)
At the start: 2 copper layers, 54.6 x 48.9 mm, 22 parts, among them J2 Conn_01x02_Female, J3 AudioJack2_SwitchT, J4 Conn_01x06_Female, J5 AudioJack2_SwitchT, SW1 SW_3PDT_x3, U101 LTC1044

Commit message: Tweak some resistor values
Parts:
- R101: value 1k -> 100
- R2: value 4.7k -> 10k
Connections:
- SW1 pad 6: Net-(SW1-Pad6) -> (no net)
- U101 pad 6: Net-(U101-Pad6) -> (no net)
- U101 pad 7: Net-(U101-Pad7) -> (no net)
Other:
- rule pad_to_mask_clearance: 0.051 -> 0
- board text added: "Switchboard r02 / NFX / Dec 2020 nuclearlighthousestudios.com"
- board text removed: "Switchboard r01 / NFX / Nov 2019 nuclearlighthousestudios.com"

Commit message: Migrate to KiCAD 6!
Other:
- net class Default removed

Commit message: Update symbols and footprints
Parts:
- J2: footprint Connector_Wire:SolderWirePad_1x02_P3.81mm_Drill1mm -> Connector_Wire:SolderWire-0.5sqmm_1x02_P4.8mm_D0.9mm_OD2.3mm
- moved J2 0.64 mm to (125.1, 71.8)
Connections:
- SW1 pad 6: (no net) -> unconnected-(SW1-Pad6)
- U101 pad 6: (no net) -> unconnected-(U101-Pad6)
- U101 pad 7: (no net) -> unconnected-(U101-Pad7)
