File: Switchboard.kicad_sch (KiCad schematic)
At the start: 16 parts, among them J2 Conn_01x02_Female, J3 AudioJack2_SwitchT, J4 Conn_01x06_Female, J5 AudioJack2_SwitchT, SW1 SW_3PDT_x3, U101 LTC1044

Commit message: Update symbols and footprints
Parts:
- C1, C103: footprint Capacitor_THT:C_Disc_D4.3mm_W1.9mm_P5.00mm -> Capacitor_THT:C_Disc_D3.0mm_W2.0mm_P2.50mm
- C101, C102, C104, C2: symbol Device:CP -> Device:C_Polarized
- J2: footprint Connector_Wire:SolderWirePad_1x02_P3.81mm_Drill1mm -> Connector_Wire:SolderWire-0.5sqmm_1x02_P4.8mm_D0.9mm_OD2.3mm
Changed lines of the file:
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@@
       (effects (font (size 1.27 1.27)) (justify left))
     )
-    (property "Footprint" "Capacitor_THT:C_Disc_D4.3mm_W1.9mm_P5.00mm" (id 2) (at 84.1502 71.755 0)
+    (property "Footprint" "Capacitor_THT:C_Disc_D3.0mm_W2.0mm_P2.50mm" (id 2) (at 84.1502 71.755 0)
       (effects (font (size 1.27 1.27)) hide)
     )
@@
     (pin "2")
   )
-  (symbol (lib_id "Device:CP") (at 94.615 67.945 0) (unit 1)
+  (symbol (lib_id "Device:C_Polarized") (at 94.615 67.945 0) (unit 1)
     (in_bom yes) (on_board yes)
     (property "Reference" "C2" (id 0) (at 97.6122 66.7766 0)
@@
       (effects (font (size 1.27 1.27)) (justify left))
     )
-    (property "Footprint" "Connector_Wire:SolderWirePad_1x02_P3.81mm_Drill1mm" (id 2) (at 56.515 66.675 0)
+    (property "Footprint" "Connector_Wire:SolderWire-0.5sqmm_1x02_P4.8mm_D0.9mm_OD2.3mm" (id 2) (at 56.515 66.675 0)
       (effects (font (size 1.27 1.27)) hide)
     )
@@
     (pin "1")
   )
-  (symbol (lib_id "Device:CP") (at 92.075 130.175 0) (unit 1)
+  (symbol (lib_id "Device:C_Polarized") (at 92.075 130.175 0) (unit 1)
     (in_bom yes) (on_board yes)
     (property "Reference" "C104" (id 0) (at 95.0722 129.0066 0)
@@
     (pin "1")
   )
-  (symbol (lib_id "Device:CP") (at 90.805 145.415 90) (unit 1)
+  (symbol (lib_id "Device:C_Polarized") (at 90.805 145.415 90) (unit 1)
     (in_bom yes) (on_board yes)
     (property "Reference" "C101" (id 0) (at 90.805 138.938 90))
@@
     (pin "2")
   )
-  (symbol (lib_id "Device:CP") (at 90.805 156.845 90) (unit 1)
+  (symbol (lib_id "Device:C_Polarized") (at 90.805 156.845 90) (unit 1)
     (in_bom yes) (on_board yes)
     (property "Reference" "C102" (id 0) (at 90.805 150.368 90))
@@
     (property "Reference" "C103" (id 0) (at 90.805 168.529 90))
     (property "Value" "100n" (id 1) (at 90.805 170.8404 90))
-    (property "Footprint" "Capacitor_THT:C_Disc_D4.3mm_W1.9mm_P5.00mm" (id 2) (at 86.995 165.4302 0)
+    (property "Footprint" "Capacitor_THT:C_Disc_D3.0mm_W2.0mm_P2.50mm" (id 2) (at 86.995 165.4302 0)
       (effects (font (size 1.27 1.27)) hide)
     )
@@
     )
     (path "/00000000-0000-0000-0000-00005bfaca48"
-      (reference "C1") (unit 1) (value "100n") (footprint "Capacitor_THT:C_Disc_D4.3mm_W1.9mm_P5.00mm")
+      (reference "C1") (unit 1) (value "100n") (footprint "Capacitor_THT:C_Disc_D3.0mm_W2.0mm_P2.50mm")
     )
     (path "/00000000-0000-0000-0000-00005bfacb00"
@@
     )
     (path "/00000000-0000-0000-0000-00005d2c1841"
-      (reference "C103") (unit 1) (value "100n") (footprint "Capacitor_THT:C_Disc_D4.3mm_W1.9mm_P5.00mm")
+      (reference "C103") (unit 1) (value "100n") (footprint "Capacitor_THT:C_Disc_D3.0mm_W2.0mm_P2.50mm")
     )
     (path "/00000000-0000-0000-0000-00005d2b3c5c"
@@
     )
     (path "/00000000-0000-0000-0000-00005bfcadb6"
-      (reference "J2") (unit 1) (value "Conn_01x02_Female") (footprint "Connector_Wire:SolderWirePad_1x02_P3.81mm_Drill1mm")
+      (reference "J2") (unit 1) (value "Conn_01x02_Female") (footprint "Connector_Wire:SolderWire-0.5sqmm_1x02_P4.8mm_D0.9mm_OD2.3mm")
     )
     (path "/00000000-0000-0000-0000-00005bfa8551"
